Commit message: Update model paths

File: model/go2.urdf (robot description, URDF)
Before this commit: robot go2_description, 41 links, 40 joints
Links:
- link FL_calf: geometry collision cylinder length=0.12 radius=0.012; visual mesh filename=package://go2_description/model/assets/calf.dae
- link FL_foot: geometry collision sphere radius=0.022; visual mesh filename=package://go2_description/model/assets/foot.dae
- link FL_hip: geometry collision cylinder length=0.04 radius=0.046; visual mesh filename=package://go2_description/model/assets/hip.dae
- link FL_thigh: geometry collision box size=0.213 0.0245 0.034; visual mesh filename=package://go2_description/model/assets/thigh.dae
- link FR_calf: geometry collision cylinder length=0.12 radius=0.013; visual mesh filename=package://go2_description/model/assets/calf_mirror.dae
- link FR_foot: geometry collision sphere radius=0.022; visual mesh filename=package://go2_description/model/assets/foot.dae
- link FR_hip: geometry collision cylinder length=0.04 radius=0.046; visual mesh filename=package://go2_description/model/assets/hip.dae
- link FR_thigh: geometry collision box size=0.213 0.0245 0.034; visual mesh filename=package://go2_description/model/assets/thigh_mirror.dae
- link RL_calf: geometry collision cylinder length=0.12 radius=0.013; visual mesh filename=package://go2_description/model/assets/calf.dae
- link RL_foot: geometry collision sphere radius=0.022; visual mesh filename=package://go2_description/model/assets/foot.dae
- link RL_hip: geometry collision cylinder length=0.04 radius=0.046; visual mesh filename=package://go2_description/model/assets/hip.dae
- link RL_thigh: geometry collision box size=0.213 0.0245 0.034; visual mesh filename=package://go2_description/model/assets/thigh.dae
- link RR_calf: geometry collision cylinder length=0.12 radius=0.013; visual mesh filename=package://go2_description/model/assets/calf_mirror.dae
- link RR_foot: geometry collision sphere radius=0.022; visual mesh filename=package://go2_description/model/assets/foot.dae
- link RR_hip: geometry collision cylinder length=0.04 radius=0.046; visual mesh filename=package://go2_description/model/assets/hip.dae
- link RR_thigh: geometry collision box size=0.213 0.0245 0.034; visual mesh filename=package://go2_description/model/assets/thigh_mirror.dae
- link base: geometry collision box size=0.3762 0.0935 0.114; visual mesh filename=package://go2_description/model/assets/base.dae

Commit message: Import collision changes back from example-robot-data

File: model/go2.urdf (robot description, URDF)
Before this commit: robot go2_description, 41 links, 40 joints
Links:
- removed link FL_calflower
- removed link FL_calflower1
- removed link FR_calflower
- removed link FR_calflower1
- removed link Head_lower
- removed link Head_upper
- removed link RL_calflower
- removed link RL_calflower1
- removed link RR_calflower
- removed link RR_calflower1
- link FL_calf: geometry collision mesh filename=package://go2_description/model/assets/collisions/calf_lowe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; collision mesh filename=package://go2_description/model/assets/collisions/calf_uppe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
- link FL_foot: geometry collision mesh filename=package://go2_description/model/assets/collisions/foot_conv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; visual mesh filename=package://go2_description/model/assets/visuals/foot.dae
- link FL_hip: geometry visual mesh filename=package://go2_description/model/assets/visuals/hip.dae
- link FL_thigh: geometry collision mesh filename=package://go2_description/model/assets/collisions/thigh_con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; visual mesh filename=package://go2_description/model/assets/visuals/thigh.dae
- link FR_calf: geometry collision mesh filename=package://go2_description/model/assets/collisions/calf_lowe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; collision mesh filename=package://go2_description/model/assets/collisions/calf_uppe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
- link FR_foot: geometry collision mesh filename=package://go2_description/model/assets/collisions/foot_conv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; visual mesh filename=package://go2_description/model/assets/visuals/foot.dae
- link FR_hip: geometry visual mesh filename=package://go2_description/model/assets/visuals/hip.dae
- link FR_thigh: geometry collision mesh filename=package://go2_description/model/assets/collisions/thigh_mir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; visual mesh filename=package://go2_description/model/assets/visuals/thigh_mirror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
- link RL_calf: geometry collision mesh filename=package://go2_description/model/assets/collisions/calf_lowe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; collision mesh filename=package://go2_description/model/assets/collisions/calf_uppe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
- link RL_foot: geometry collision mesh filename=package://go2_description/model/assets/collisions/foot_conv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; visual mesh filename=package://go2_description/model/assets/visuals/foot.dae
- link RL_hip: geometry collision mesh filename=package://go2_description/model/assets/collisions/hip_conve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; visual mesh filename=package://go2_description/model/assets/visuals/hip.dae
- link RL_thigh: geometry collision mesh filename=package://go2_description/model/assets/collisions/thigh_con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; visual mesh filename=package://go2_description/model/assets/visuals/thigh.dae
- link RR_calf: geometry collision mesh filename=package://go2_description/model/assets/collisions/calf_lowe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; collision mesh filename=package://go2_description/model/assets/collisions/calf_uppe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
- link RR_foot: geometry collision mesh filename=package://go2_description/model/assets/collisions/foot_conv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; visual mesh filename=package://go2_description/model/assets/visuals/foot.dae
- link RR_hip: geometry collision mesh filename=package://go2_description/model/assets/collisions/hip_conve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; visual mesh filename=package://go2_description/model/assets/visuals/hip.dae
- link RR_thigh: geometry collision mesh filename=package://go2_description/model/assets/collisions/thigh_mir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; visual mesh filename=package://go2_description/model/assets/visuals/thigh_mirror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
- link base: geometry collision mesh filename=package://go2_description/model/assets/collisions/base_conv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; visual mesh filename=package://go2_description/model/assets/visuals/base.dae
Joints:
- removed joint FL_calflower1_joint
- removed joint FL_calflower_joint
- removed joint FR_calflower1_joint
- removed joint FR_calflower_joint
- removed joint Head_lower_joint
- removed joint Head_upper_joint
- removed joint RL_calflower1_joint
- removed joint RL_calflower_joint
- removed joint RR_calflower1_joint
- removed joint RR_calflower_joint
